File: MKRShield_v1.kicad_pcb (KiCad board)
At the start: 4 copper layers, 67.6 x 25 mm, 11 parts, among them J3 DNP, J5 DNP

Commit message: fix default pins for kicad 5
Parts:
- removed J3, J5: DNP, MKRFoxShield_v2:1X14_SMD_TH
- added J1: , Pines:61301411121, F.Cu at (153.2, 115.2)
- added J2: , Pines:61301411121, F.Cu at (153.2, 94.8)
Other:
- board text removed: "X1"
